File: PCB/WeatherStationPCB/WeatherStationPCB.kicad_pcb (KiCad board)
At the start: 4 copper layers, 104.1 x 92.5 mm, 36 parts, among them J1 Conn_01x06_Male, J2 Conn_01x06_Male, J3 Conn_01x20_Pin, J4 Conn_01x20_Pin, J5 Conn_01x03_Pin, J6 Conn_01x05_Socket, J7 Conn_01x06_Pin, J8 Conn_01x06_Pin, Q1 2N7000, Q2 2N7000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

Commit message: Move data to new JSON format
Parts:
- added R8: 23GR, Resistor_THT:R_Axial_DIN0207_L6.3mm_D2.5mm_P10.16mm_Horizontal, F.Cu at (187.8, 112.0)
- added R9: 23GR, Resistor_THT:R_Axial_DIN0207_L6.3mm_D2.5mm_P10.16mm_Horizontal, F.Cu at (177.6, 108.5)
Connections:
- U2 pad 1: /RTC_BAT -> Net-(U2-BAT)
Routing:
- net GND: track 402.2 -> 421.4 mm
- net /RTC_BAT: track 18.6 -> 37.1 mm
- net Net-(U2-BAT): track 0.00 -> 7.11 mm
